Commit message: update scanning from zed

File: ur10e_zed_moveit_config/zed_description/urdf/ur10e_zed_macro.xacro (robot description, xacro)
@@ -17,5 +17,5 @@
           real robot.
   -->
-  <xacro:macro name="ur10e_ka_robot" params="
+  <xacro:macro name="ur10e_zed_robot" params="
    prefix
    joint_limits_parameters_file:='$(find ur_description)/config/ur10e/joint_limits.yaml'
@@ -40,5 +40,5 @@
       safety_k_position="${safety_k_position}"
     />
-    <xacro:include filename="$(find ur10e_ka_moveit_config)/ka_description/urdf/ka_macro.xacro"/>
+    <xacro:include filename="$(find ur10e_zed_moveit_config)/zed_description/urdf/zed_macro.xacro"/>
     <xacro:end_effector prefix="" connected_to="flange"/>
   </xacro:macro>
